File: Hardware/Schematic_tema.brd (EAGLE design)
At the start: 46 x 35 mm, 105 parts, among them IC1 BQ25180YBGR, IC2 DRV2605YZFR, IC3 BMA421, IC9 RT6160AWSC, J1 503480-2400, J2 TC2030-IDC, J4 KH-TYPE-C-16P, Q1 20V/4.2A/52mΩ/1.4W, Q3 SI1308EDL-T1-GE3, U1 NRF52840_QF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

Commit message: Updated the entire project
Parts:
- moved R_TYPE_SEL 1.95 mm to (25.1, 38.7)
- moved R3 1.13 mm to (28.5, 31.0)
- moved R1_EP_DR 0.38 mm to (24.6, 34.0)
- moved D3 0.18 mm to (37.1, 34.9)
- moved R17 0.16 mm to (30.0, 30.0)
- moved L2 0.15 mm to (35.2, 34.5)
- moved TP_SDA 0.15 mm to (36.9, 22.4)
- moved R9 0.06 mm to (35.3, 22.5)
Connections:
- removed net N$20: Q3.1, R2_EP_DR.2
- net GDR: now also Q3.1, R2_EP_DR.2
Routing:
- net GND: track 178.2 -> 169.9 mm
- net GDR: track 0.00 -> 4.71 mm, vias 0 -> 2
- net VREG: track 17.2 -> 15.3 mm
- net N$21: track 10.1 -> 11.8 mm
- net N$20: track 1.05 -> 0.00 mm
- net EPD_3V3: track 54.2 -> 55.1 mm
- net N$1: track 1.21 -> 1.97 mm
- net VBAT/2.5C: track 6.19 -> 6.94 mm
- net SDA/2.4C: track 29.1 -> 29.8 mm
- net RESE: track 5.56 -> 6.09 mm
- net 3V3/2.4A: track 119.7 -> 120.2 mm, vias 16 -> 18
Other:
- outline, holes or cut-outs redrawn
