File: Hardware/Schematic_tema.sch (EAGLE design)
At the start: 105 parts, among them IC1 BQ25180YBGR, IC2 DRV2605YZFR, IC3 BMA421, IC9 RT6160AWSC, J1 503480-2400, J2 TC2030-IDC, J4 KH-TYPE-C-16P, Q1 20V/4.2A/52mΩ/1.4W, Q3 SI1308EDL-T1-GE3, U1 NRF52840_QF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

Commit message: Updated the entire project
Connections:
- removed net N$20: Q3.G, R2_EP_DR.2
- net GDR: now also Q3.G, R2_EP_DR.2
Other:
- note added: "DEC1"
